Commit message: rmpflow config file modifing

File: config/RMPFlow.urdf (robot description, URDF)
Before this commit: robot ur10, 9 links, 8 joints
Links:
- removed link ee_link
- removed link forearm_link
- removed link shoulder_link
- removed link upper_arm_link
- removed link wrist_1_link
- removed link wrist_2_link
- removed link wrist_3_link
- added link finger_width
- added link joint_1
- added link joint_2
- added link joint_3
- added link joint_4
- added link joint_5
- added link joint_6
Joints:
- joint ee_joint: parent wrist_3_link -> joint_6
- joint elbow_joint: child forearm_link -> joint_3; parent upper_arm_link -> joint_2
- joint shoulder_lift_joint: child upper_arm_link -> joint_2; parent shoulder_link -> joint_1
- joint shoulder_pan_joint: child shoulder_link -> joint_1
- joint wrist_1_joint: child wrist_1_link -> joint_4; parent forearm_link -> joint_3
- joint wrist_2_joint: child wrist_2_link -> joint_5; parent wrist_1_link -> joint_4
- joint wrist_3_joint: child wrist_3_link -> joint_6; parent wrist_2_link -> joint_5
